Commit message: bug fix

File: jy_bot/urdf/jy_bot.xacro (robot description, xacro)
@@ -159,5 +159,5 @@
       <origin xyz="0 0 0" rpy="0 0 0"/>
       <geometry>
-        <mesh filename="package://udacity_bot/meshes/hokuyo.dae"/>
+        <mesh filename="package://jy_bot/meshes/hokuyo.dae"/>
       </geometry>
     </visual>
